File: Hardware/Weatherever_board_rev1/USB_Dongle.kicad_sch (KiCad schematic)
At the start: 34 parts, among them J101 USB_B_Micro, J103 Test pins COMM1, J104 DebugConn, J106 Test pins COMM2, SW102 RESET, U101 USBLC6-2P6, U102 FT230XQ, U103 AOZ1312, U104 NCP115AMX250TCG, U105 STM32G030C8T6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

Commit message: Layout impl start
Parts:
- removed SW102: RESET, symbol Switch:SW_MEC_5E
- removed Y101: 49S-16.000MEEJ-T 16MHz, symbol Device:Crystal
- added SW102: RESET, Button_Switch_SMD:SW_Push_1P1T_NO_6x6mm_H9.5mm, symbol Switch:SW_Push
- added Y101: 3225-16M-SR 16MHz 9pF, Crystal:Crystal_SMD_TXC_7M-4Pin_3.2x2.5mm_HandSoldering, symbol Device:Crystal_GND24
- D101, D102, D103: footprint (none) -> Diode_SMD:D_0805_2012Metric_Pad1.15x1.40mm_HandSolder
- Y102: footprint (none) -> Crystal:Crystal_SMD_TXC_7A-2Pin_5x3.2mm
Connections:
- net GNDD: now also SW102.1, Y101.2, Y101.4
- net HF_OSC_IN: now also Y101.3
- net HF_OSC_OUT: now also Y101.1
- net ~{RESET}: now also SW102.2
