File: Hardware/Giskard_rev1/GiskardRF/ExpansionConnector.kicad_sch (KiCad schematic)
At the start: 14 parts, among them J107 Conn_02x05_Odd_Even, U108 AP22802AW5-7, U4 USBLC6-4SC6

Commit message: layout dev
Connections:
- net CONTACT_PWR: now also J107.4 (Pin_4), J107.6 (Pin_6); no longer J107.2 (Pin_2), J107.2 (Pin_2), J107.2 (Pin_2)
- net GNDD: now also J107.2 (Pin_2), J107.2 (Pin_2), J107.2 (Pin_2); no longer J107.4 (Pin_4), J107.6 (Pin_6)
Changed lines of the file:
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@@
   (junction (at 219.075 102.87) (diameter 0) (color 0 0 0 0)
   )
+  (junction (at 136.525 45.72) (diameter 0) (color 0 0 0 0)
+  )
   (junction (at 181.61 45.72) (diameter 0) (color 0 0 0 0)
   )
+  (junction (at 88.265 45.72) (diameter 0) (color 0 0 0 0)
+  )
+  (junction (at 225.425 45.085) (diameter 0) (color 0 0 0 0)
+  )
   (junction (at 190.5 102.87) (diameter 0) (color 0 0 0 0)
   )
   (junction (at 208.28 52.705) (diameter 0) (color 0 0 0 0)
   )
-  (junction (at 136.525 45.72) (diameter 0) (color 0 0 0 0)
-  )
   (junction (at 194.31 114.3) (diameter 0) (color 0 0 0 0)
   )
@@
     (stroke (width 0) (type default))
   )
-  (wire (pts (xy 234.315 45.085) (xy 223.52 45.085))
+  (wire (pts (xy 234.315 45.085) (xy 225.425 45.085))
     (stroke (width 0) (type default))
   )
@@
     (stroke (width 0) (type default))
   )
+  (wire (pts (xy 136.525 43.18) (xy 135.255 43.18))
+    (stroke (width 0) (type default))
+  )
   (wire (pts (xy 72.39 45.72) (xy 73.66 45.72))
     (stroke (width 0) (type default))
   )
-  (wire (pts (xy 136.525 43.18) (xy 135.255 43.18))
-    (stroke (width 0) (type default))
-  )
   (wire (pts (xy 190.5 101.6) (xy 190.5 102.87))
     (stroke (width 0) (type default))
@@
     (stroke (width 0) (type default))
   )
+  (wire (pts (xy 136.525 45.72) (xy 136.525 43.18))
+    (stroke (width 0) (type default))
+  )
   (wire (pts (xy 179.705 48.26) (xy 181.61 48.26))
     (stroke (width 0) (type default))
@@
     (stroke (width 0) (type default))
   )
+  (wire (pts (xy 138.43 45.72) (xy 136.525 45.72))
+    (stroke (width 0) (type default))
+  )
   (wire (pts (xy 130.175 116.84) (xy 130.81 116.84))
     (stroke (width 0) (type default))
@@
     (stroke (width 0) (type default))
   )
-  (wire (pts (xy 224.155 42.545) (xy 223.52 42.545))
+  (wire (pts (xy 223.52 42.545) (xy 225.425 42.545))
     (stroke (width 0) (type default))
   )
@@
     (stroke (width 0) (type default))
   )
+  (wire (pts (xy 135.255 45.72) (xy 136.525 45.72))
+    (stroke (width 0) (type default))
+  )
   (wire (pts (xy 102.235 87.63) (xy 104.14 87.63))
     (stroke (width 0) (type default))
   )
-  (wire (pts (xy 86.36 45.72) (xy 98.425 45.72))
+  (wire (pts (xy 86.36 45.72) (xy 88.265 45.72))
     (stroke (width 0) (type default))
   )
@@
     (stroke (width 0) (type default))
   )
+  (wire (pts (xy 181.61 43.18) (xy 181.61 45.72))
+    (stroke (width 0) (type default))
+  )
   (wire (pts (xy 121.92 53.34) (xy 122.555 53.34))
     (stroke (width 0) (type default))
   )
+  (wire (pts (xy 225.425 42.545) (xy 225.425 45.085))
+    (stroke (width 0) (type default))
+  )
   (wire (pts (xy 129.54 144.145) (xy 130.175 144.145))
     (stroke (width 0) (type default))
   )
-  (wire (pts (xy 86.36 43.18) (xy 86.995 43.18))
+  (wire (pts (xy 86.36 43.18) (xy 88.265 43.18))
     (stroke (width 0) (type default))
   )
@@
     (stroke (width 0) (type default))
   )
-  (wire (pts (xy 135.255 45.72) (xy 136.525 45.72))
-    (stroke (width 0) (type default))
-  )
   (wire (pts (xy 184.785 118.11) (xy 204.47 118.11))
     (stroke (width 0) (type default))
@@
     (stroke (width 0) (type default))
   )
-  (wire (pts (xy 136.525 45.72) (xy 146.05 45.72))
-    (stroke (width 0) (type default))
-  )
   (wire (pts (xy 80.645 82.55) (xy 81.915 82.55))
     (stroke (width 0) (type default))
@@
     (stroke (width 0) (type default))
   )
+  (wire (pts (xy 88.265 43.18) (xy 88.265 45.72))
+    (stroke (width 0) (type default))
+  )
   (wire (pts (xy 150.495 139.065) (xy 151.13 139.065))
     (stroke (width 0) (type default))
@@
     (stroke (width 0) (type default))
   )
-  (wire (pts (xy 180.34 43.18) (xy 179.705 43.18))
+  (wire (pts (xy 179.705 43.18) (xy 181.61 43.18))
     (stroke (width 0) (type default))
   )
@@
     (stroke (width 0) (type default))
   )
+  (wire (pts (xy 88.265 45.72) (xy 98.425 45.72))
+    (stroke (width 0) (type default))
+  )
   (wire (pts (xy 151.765 116.84) (xy 151.13 116.84))
     (stroke (width 0) (type default))
@@
   )
   (wire (pts (xy 166.37 53.34) (xy 167.005 53.34))
+    (stroke (width 0) (type default))
+  )
+  (wire (pts (xy 225.425 45.085) (xy 223.52 45.085))
     (stroke (width 0) (type default))
   )
@@
     (effects (font (size 2 2) (thickness 0.508) bold) (justify left bottom))
   )
-  (label "CONTACT_PWR" (at 180.34 43.18 0) (fields_autoplaced)
-    (effects (font (size 1.27 1.27)) (justify left bottom))
-  )
   (label "CONTACT_PWR" (at 93.345 130.81 0) (fields_autoplaced)
     (effects (font (size 1.27 1.27)) (justify left bottom))
   )
-  (label "CONTACT_PWR" (at 136.525 43.18 0) (fields_autoplaced)
+  (label "CONTACT_PWR" (at 138.43 45.72 0) (fields_autoplaced)
     (effects (font (size 1.27 1.27)) (justify left bottom))
   )
@@
   (label "CONTACT_PWR" (at 190.5 101.6 180) (fields_autoplaced)
     (effects (font (size 1.27 1.27)) (justify right bottom))
-  )
-  (label "CONTACT_PWR" (at 224.155 42.545 0) (fields_autoplaced)
-    (effects (font (size 1.27 1.27)) (justify left bottom))
-  )
-  (label "CONTACT_PWR" (at 86.995 43.18 0) (fields_autoplaced)
-    (effects (font (size 1.27 1.27)) (justify left bottom))
   )
   (label "CONTACT_PWR" (at 142.24 74.295 0) (fields_autoplaced)
@@
         )
       )
-      (project "Weatherever_board_rev1"
-        (path "/e63e39d7-6ac0-4ffd-8aa3-1841a4541b55"
-          (reference "#PWR0122") (unit 1)
-        )
-        (path "/e63e39d7-6ac0-4ffd-8aa3-1841a4541b55/d4942633-f47c-4824-8407-5ebb1716d5e1"
-          (reference "#PWR0622") (unit 1)
-        )
-      )
-    )
-  )
-  (symbol (lib_id "power:GNDD") (at 146.05 45.72 90) (unit 1)
-    (in_bom yes) (on_board yes) (dnp no)
-    (property "Reference" "#PWR0122" (at 152.4 45.72 0)
-      (effects (font (size 1.27 1.27)) hide)
-    )
-    (property "Value" "GNDD" (at 149.225 48.26 0)
-      (effects (font (size 1.27 1.27)) (justify left))
-    )
-    (property "Footprint" "" (at 146.05 45.72 0)
-      (effects (font (size 1.27 1.27)) hide)
-    )
-    (property "Datasheet" "" (at 146.05 45.72 0)
-      (effects (font (size 1.27 1.27)) hide)
-    )
-    (pin "1")
-    (instances
-      (project "USB_Dongle"
-        (path "/361e19cb-cc91-422e-84ec-3a573b4fa89d"
-          (reference "#PWR0122") (unit 1)
-        )
-      )
-      (project "GiskardRF"
-        (path "/e1ed0ee6-e1ed-4994-9bff-2a49a44995c0"
-          (reference "#PWR0141") (unit 1)
-        )
-        (path "/e1ed0ee6-e1ed-4994-9bff-2a49a44995c0/e974328c-811c-4ed4-a726-e121a6085980"
-          (reference "#PWR0303") (unit 1)
-        )
-      )

Commit message: layout dev part 2
Parts:
- removed U4 (x6): USBLC6-4SC6, Package_TO_SOT_SMD:SOT-23-6, symbol Power_Protection:USBLC6-4SC6
Connections:
- net GNDD: now also J107.1 (Pin_1), J107.10 (Pin_10), J107.3 (Pin_3), J107.3 (Pin_3), J107.6 (Pin_6), J107.8 (Pin_8); no longer J107.2 (Pin_2), J107.2 (Pin_2), J107.2 (Pin_2), J107.4 (Pin_4), J107.4 (Pin_4), J107.5 (Pin_5), J107.5 (Pin_5), J107.9 (Pin_9)
- net GPIO_PA0: now also J107.5 (Pin_5); no longer J107.1 (Pin_1)
- net GPIO_PA1: now also J107.4 (Pin_4); no longer J107.3 (Pin_3)
- net GPIO_PA2: now also J107.2 (Pin_2); no longer J107.7 (Pin_7)
- net GPIO_PA3: now also J107.1 (Pin_1); no longer J107.9 (Pin_9)
- net GPIO_PA4: now also J107.3 (Pin_3); no longer J107.6 (Pin_6)
- net GPIO_PA8: now also J107.10 (Pin_10); no longer J107.8 (Pin_8)
- net GPIO_PB15: now also J107.8 (Pin_8); no longer J107.10 (Pin_10)
- net GPIO_PB3: now also J107.9 (Pin_9); no longer J107.9 (Pin_9)
- net GPIO_PB4: now also J107.10 (Pin_10); no longer J107.10 (Pin_10)
- net GPIO_PB5: now also J107.8 (Pin_8); no longer J107.8 (Pin_8)
- net GPIO_PB8: now also J107.6 (Pin_6); no longer J107.1 (Pin_1)
- net GPIO_PB9: now also J107.4 (Pin_4); no longer J107.3 (Pin_3)
- net GPIO_PC13: now also J107.2 (Pin_2); no longer J107.10 (Pin_10)
- net GPIO_PC6: now also J107.9 (Pin_9); no longer J107.6 (Pin_6)
- net GPIO_PC7: now also J107.7 (Pin_7); no longer J107.8 (Pin_8)
- net GPIO_PD3: now also J107.1 (Pin_1); no longer J107.7 (Pin_7)
- net I2C1_SCL: now also J107.2 (Pin_2); no longer J107.1 (Pin_1)
- net I2C1_SDA: now also J107.10 (Pin_10); no longer J107.3 (Pin_3)
- net SPI1_MISO: now also J107.7 (Pin_7); no longer J107.9 (Pin_9)
- net SPI1_MOSI: now also J107.9 (Pin_9); no longer J107.10 (Pin_10)
- net SPI1_SCK: now also J107.5 (Pin_5); no longer J107.7 (Pin_7)
- net CONTACT_PWR renamed CON_PWR
- new net GPIO_PB13: J107.7 (Pin_7)
- new net GPIO_PB14: J107.9 (Pin_9)
Other:
- moved on the sheet: C105, R108, U108

Commit message: Layout dev part 3
Parts:
- removed J107 (x4): Conn_02x05_Odd_Even, Connector_PinHeader_1.27mm:PinHeader_2x05_P1.27mm_Vertical_SMD, symbol Connector_Generic:Conn_02x05_Odd_Even
- added J305, J306: Conn_01x16, Connector_PinHeader_2.54mm:PinHeader_1x16_P2.54mm_Vertical_SMD_Pin1Left, symbol Connector_Generic:Conn_01x16
Connections:
- net CON_PWR: now also J305.16 (Pin_16), J306.1 (Pin_1)
- net GNDD: now also J305.1 (Pin_1), J305.2 (Pin_2), J306.15 (Pin_15), J306.16 (Pin_16)
- net GPIO_PA0: now also J305.10 (Pin_10)
- net GPIO_PA1: now also J305.9 (Pin_9)
- net GPIO_PA2: now also J305.8 (Pin_8)
- net GPIO_PA3: now also J305.3 (Pin_3)
- net GPIO_PA4: now also J305.4 (Pin_4)
- net GPIO_PA8: now also J305.11 (Pin_11)
- net GPIO_PB13: now also J305.14 (Pin_14)
- net GPIO_PB14: now also J305.13 (Pin_13)
- net GPIO_PB15: now also J305.12 (Pin_12)
- net GPIO_PB3: now also J306.10 (Pin_10)
- net GPIO_PB4: now also J306.14 (Pin_14)
- net GPIO_PB5: now also J305.15 (Pin_15)
- net GPIO_PB8: now also J306.13 (Pin_13)
- net GPIO_PB9: now also J306.12 (Pin_12)
- net GPIO_PC13: now also J306.11 (Pin_11)
- net GPIO_PC6: now also J306.6 (Pin_6)
- net GPIO_PC7: now also J306.5 (Pin_5)
- net GPIO_PD0: now also J306.2 (Pin_2)
- net GPIO_PD1: now also J306.3 (Pin_3)
- net GPIO_PD2: now also J306.4 (Pin_4)
- net GPIO_PD3: now also J306.9 (Pin_9)
- net I2C1_SCL: now also J306.7 (Pin_7)
- net I2C1_SDA: now also J306.8 (Pin_8)
- net SPI1_MISO: now also J305.6 (Pin_6)
- net SPI1_MOSI: now also J305.7 (Pin_7)
- net SPI1_SCK: now also J305.5 (Pin_5)
Other:
- moved on the sheet: C105, R108, U108

Commit message: Finished Giskard layout
- Need to fix DRC violations
- It'd be nice to move EEPROM closer to MPU
Parts:
- J305: value Conn_01x16 -> Conn_01x14; footprint Connector_PinHeader_2.54mm:PinHeader_1x16_P2.54mm_Vertical_SMD_Pin1Left -> Connector_PinHeader_2.54mm:PinHeader_1x14_P2.54mm_Vertical; symbol Connector_Generic:Conn_01x16 -> Connector_Generic:Conn_01x14
- J306: footprint Connector_PinHeader_2.54mm:PinHeader_1x16_P2.54mm_Vertical_SMD_Pin1Left -> Connector_PinHeader_2.54mm:PinHeader_1x16_P2.54mm_Vertical
Connections:
- net GPIO_PB8 is gone; now on net I2C1_SCL: J306.13 (Pin_13)
- net GPIO_PB9 is gone; now on net GPIO_PB5: J306.12 (Pin_12)
- net GPIO_PC13 is gone; now on net GPIO_PB4: J306.11 (Pin_11)
- net GPIO_PD0 is gone; now on net CON_PWR: J306.2 (Pin_2)
- net GPIO_PD2 is gone; now on net GPIO_PB13: J306.4 (Pin_4)
- net GPIO_PD3 is gone; now on net GPIO_PC7: J306.9 (Pin_9)
- net CON_PWR: no longer J305.16 (Pin_16)
- net GNDD: now also J305.14 (Pin_14); no longer J305.1 (Pin_1), J305.2 (Pin_2)
- net GPIO_PA0: now also J305.1 (Pin_1); no longer J305.10 (Pin_10)
- net GPIO_PA1: now also J305.2 (Pin_2); no longer J305.9 (Pin_9)
- net GPIO_PA2: now also J305.3 (Pin_3); no longer J305.8 (Pin_8)
- net GPIO_PA3: now also J305.4 (Pin_4); no longer J305.3 (Pin_3)
- net GPIO_PA4: now also J305.5 (Pin_5); no longer J305.4 (Pin_4)
- net GPIO_PA8: now also J306.7 (Pin_7); no longer J305.11 (Pin_11)
- net GPIO_PB13: no longer J305.14 (Pin_14)
- net GPIO_PB14: now also J306.5 (Pin_5); no longer J305.13 (Pin_13)
- net GPIO_PB15: now also J306.6 (Pin_6); no longer J305.12 (Pin_12)
- net GPIO_PB4: no longer J306.14 (Pin_14)
- net GPIO_PB5: no longer J305.15 (Pin_15)
- net GPIO_PC6: now also J306.8 (Pin_8); no longer J306.6 (Pin_6)
- net GPIO_PC7: no longer J306.5 (Pin_5)
- net I2C1_SCL: no longer J306.7 (Pin_7)
- net I2C1_SDA: now also J306.14 (Pin_14); no longer J306.8 (Pin_8)
- net SPI1_MISO: now also J305.7 (Pin_7); no longer J305.6 (Pin_6)
- net SPI1_MOSI: now also J305.8 (Pin_8); no longer J305.7 (Pin_7)
- net SPI1_SCK: now also J305.6 (Pin_6); no longer J305.5 (Pin_5)
- net GPIO_PD1 renamed GPIO_PB12
- new net GPIO_PB0: J305.9 (Pin_9)
- new net GPIO_PB1: J305.10 (Pin_10)
- new net GPIO_PB10: J305.12 (Pin_12)
- new net GPIO_PB11: J305.13 (Pin_13)
- new net GPIO_PB2: J305.11 (Pin_11)
