File: Hardware/Giskard_rev1/GiskardRF/GiskardRF.kicad_sch (KiCad schematic)
At the start: 50 parts, among them J101 USB_B_Micro, J103 Test pins COMM1, J104 DebugConn, J105 ExtensionConn, J106 Test pins COMM2, SW102 RESET, U101 USBLC6-2P6, U102 FT230XQ, U103 AP22802AW5-7, U105 STM32G030C8T6, U106 M24C16-RM, U107 23K256-I/SN, U108 AP22802AW5-7, U110 AP2127K-3.3, Y101 3225-16M-SR 16MHz 9pF, Y102 32.768K-CFPX217

Commit message: Upgrade to stmg07
Parts:
- removed C116: 100n, Capacitor_SMD:C_0805_2012Metric_Pad1.18x1.45mm_HandSolder, symbol Device:C_Small
- removed R105: 1k, Resistor_SMD:R_0805_2012Metric_Pad1.20x1.40mm_HandSolder, symbol Device:R_Small
- removed U107: 23K256-I/SN, Package_SO:SO-8_3.9x4.9mm_P1.27mm, symbol CustomSymbols:23K256-I/SN
- added U104: STM32G070CBTx, Package_QFP:LQFP-48_7x7mm_P0.5mm, symbol MCU_ST_STM32G0:STM32G070CBTx
- C112, C113: value 100n -> 20p
- C114, C115: value 100n -> 13p
- Y102: footprint Crystal:Crystal_SMD_TXC_7A-2Pin_5x3.2mm -> Crystal:Crystal_SMD_MicroCrystal_CC7V-T1A-2Pin_3.2x1.5mm_HandSoldering
Other:
- note added: "ZAMIENIC NA G07"
- note removed: "General purpose SRAM"
- moved on the sheet: C105, C107, C108, J103, J105, J106, R108, R109, R110, R111, U105, U108

Commit message: Layout development 1
Parts:
- added BT1: RTC_Bat, Battery:BatteryHolder_Keystone_3002_1x2032, symbol Device:Battery_Cell
- added C1, C108: 100n, Capacitor_SMD:C_0805_2012Metric_Pad1.18x1.45mm_HandSolder, symbol Device:C_Small
- added C107: 10u, Capacitor_SMD:C_0805_2012Metric_Pad1.18x1.45mm_HandSolder, symbol Device:C_Small
- added J1: Conn_ARM_JTAG_SWD_20, Connector_IDC:IDC-Header_2x10_P2.54mm_Horizontal, symbol Connector:Conn_ARM_JTAG_SWD_20
- added R1, R2, R3, R4: 3k3, Resistor_SMD:R_0805_2012Metric_Pad1.20x1.40mm_HandSolder, symbol Device:R_Small
- added U3: USBLC6-4SC6, Package_TO_SOT_SMD:SOT-23-6, symbol Power_Protection:USBLC6-4SC6
- J105: value ExtensionConn -> DS1020-07-20VBT1B; footprint Connector_IDC:IDC-Header_2x10_P2.54mm_Horizontal -> Connector_FFC-FPC:TE_2-84952-0_1x20-1MP_P1.0mm_Horizontal; symbol Connector_Generic:Conn_02x10_Odd_Even -> Connector_Generic:Conn_01x20
Connections:
- net +3V3: now also U104.5 (VREF+), U104.6 (VDD), C107.1, C108.1, R1.1, R2.1, R3.1, R4.1
- net 3V_Bat: now also U104.4 (VBAT), BT1.1 (+), C1.1
- net CONN_PWR: now also U3.5 (VBUS)
- net GNDD: now also J105.5 (Pin_5), J105.9 (Pin_9), U104.7 (VSS), BT1.2 (-), C1.2, C107.2, C108.2, U3.2 (GND); no longer J105.4 (Pin_4), J105.8 (Pin_8)
- net GPIO_A1: now also U104.12 (PA1)
- net GPIO_A15: now also J105.13 (Pin_13); no longer J105.6 (Pin_6)
- net GPIO_A2: now also U104.13 (PA2)
- net GPIO_A8: now also U104.28 (PA8)
- net GPIO_B15: now also U104.27 (PB15), U104.37 (PA15)
- net GPIO_B3: now also J105.14 (Pin_14), U104.42 (PB3); no longer J105.10 (Pin_10)
- net GPIO_B4: now also J105.15 (Pin_15), U104.43 (PB4); no longer J105.12 (Pin_12)
- net GPIO_B5: now also J105.16 (Pin_16), U104.44 (PB5); no longer J105.14 (Pin_14)
- net GPIO_B8: now also J105.17 (Pin_17), U104.47 (PB8); no longer J105.16 (Pin_16)
- net GPIO_B9: now also U104.48 (PB9)
- net GPIO_C13: now also U104.1 (PC13)
- net GPIO_C6: now also U104.30 (PC6)
- net GPIO_C7: now also U104.31 (PC7)
- net GPIO_D1: now also J105.10 (Pin_10), U104.39 (PD1); no longer J105.13 (Pin_13)
- net GPIO_D2: now also J105.11 (Pin_11), U104.40 (PD2); no longer J105.15 (Pin_15)
- net GPIO_D3: now also J105.12 (Pin_12), U104.41 (PD3); no longer J105.17 (Pin_17)
- net HF_OSC_IN: now also U104.8 (PF0)
- net HF_OSC_OUT: now also U104.9 (PF1)
- net I2C1_SCL: now also J105.4 (Pin_4), U104.29 (PA9/NC), R1.2, U3.4 (I/O3); no longer J105.5 (Pin_5)
- net I2C1_SDA: now also U104.32 (PA10/NC), R2.2, U3.6 (I/O4)
- net I2C2_SCL_MEM: now also U104.25 (PB13), R3.2
- net I2C2_SDA_MEM: now also U104.26 (PB14), R4.2
- net LF_OSC_IN: now also U104.2 (PC14)
- net LF_OSC_OUT: now also U104.3 (PC15)
- net RF_DIO_0: now also U104.19 (PB0)
- net RF_DIO_1: now also U104.20 (PB1)
- net RF_DIO_2: now also U104.21 (PB2)
- net RF_DIO_3: now also U104.22 (PB10)
- net RF_DIO_4: now also U104.23 (PB11)
- net RF_DIO_5: now also U104.24 (PB12)
- net SPI1_MISO: now also J105.7 (Pin_7), U104.17 (PA6); no longer J105.9 (Pin_9)
- net SPI1_MOSI: now also J105.8 (Pin_8), U104.18 (PA7); no longer J105.11 (Pin_11)
- net SPI1_SCK: now also J105.6 (Pin_6), U104.16 (PA5); no longer J105.7 (Pin_7)
- net SPI2_MISO: now also U104.14 (PA3)
- net SPI2_MOSI: now also U104.15 (PA4)
- net SPI2_SCK: now also U104.11 (PA0)
- net SW_CLK: now also U104.36 (PA14)
- net SW_DIO: now also U104.35 (PA13)
- net USART1_CTS: now also U104.33 (PA11/PA9)
- net USART1_RTS: now also U104.34 (PA12/PA10)
- net USART1_RX: now also U104.46 (PB7)
- net USART1_TX: now also U104.45 (PB6)
- net ~{ERR_LED}: now also U104.38 (PD0)
- net ~{RESET}: now also U104.10 (NRST)
- new net: J1.10 (GND), J1.12 (GND), J1.14 (GND), J1.16 (GND), J1.18 (GND), J1.20 (GND), J1.4 (GND), J1.6 (GND), J1.8 (GND)
Other:
- note added: "ESD protection"
- note removed: "Extension connector"
- moved on the sheet: C105, C107, C108, J103, J105, J106, R108, R109, R110, R111, U104, U105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

Commit message: Board dev + new sw target
Parts:
- removed J1: Conn_ARM_JTAG_SWD_20, Connector_IDC:IDC-Header_2x10_P2.54mm_Horizontal, symbol Connector:Conn_ARM_JTAG_SWD_20
- removed J104: DebugConn, Connector_IDC:IDC-Header_2x03_P2.54mm_Vertical, symbol Connector_Generic:Conn_01x06
- added J2: Conn_ARM_JTAG_SWD_20, Connector_IDC:IDC-Header_2x10_P2.54mm_Horizontal, symbol Connector:Conn_ARM_JTAG_SWD_20
- added U1, U2, U4: USBLC6-4SC6, Package_TO_SOT_SMD:SOT-23-6, symbol Power_Protection:USBLC6-4SC6
Connections:
- net +3V3: now also J2.1 (VTREF), J2.2 (VCC/NC)
- net CONN_PWR: now also U1.5 (VBUS), U2.5 (VBUS), U4.5 (VBUS)
- net GNDD: now also J2.10 (GND), J2.12 (GND), J2.13 (TDO/SWO), J2.14 (GND), J2.16 (GND), J2.18 (GND), J2.20 (GND), J2.3 (~{TRST}), J2.4 (GND), J2.5 (TDI), J2.6 (GND), J2.8 (GND), U1.2 (GND), U2.2 (GND), U4.2 (GND)
- net GPIO_A15: now also U1.1 (I/O1)
- net GPIO_B3: now also U4.3 (I/O2)
- net GPIO_B4: now also U2.1 (I/O1)
- net GPIO_B5: now also U2.3 (I/O2)
- net GPIO_B8: now also U2.6 (I/O4)
- net GPIO_B9: now also U2.4 (I/O3)
- net GPIO_D1: now also U1.6 (I/O4)
- net GPIO_D2: now also U1.4 (I/O3)
- net GPIO_D3: now also U1.3 (I/O2)
- net I2C2_SCL_MEM: now also J106.4 (Pin_4)
- net I2C2_SDA_MEM: now also J106.3 (Pin_3)
- net SPI1_MISO: no longer J103.4 (Pin_4)
- net SPI1_MOSI: now also U3.3 (I/O2); no longer J103.3 (Pin_3)
- net SPI1_SCK: now also U3.1 (I/O1); no longer J103.5 (Pin_5)
- net SPI2_MISO: now also J103.3 (Pin_3)
- net SPI2_MOSI: now also J103.4 (Pin_4)
- net SPI2_SCK: now also J103.5 (Pin_5)
- net SW_CLK: now also J2.9 (TCK/SWDCLK), U4.4 (I/O3)
- net SW_DIO: now also J2.7 (TMS/SWDIO), U4.1 (I/O1)
- net USART1_CTS: no longer J106.4 (Pin_4)
- net USART1_RTS: no longer J106.3 (Pin_3)
- net ~{RESET}: now also J2.15 (~{SRST})
- no-connect marks 4 -> 8
Other:
- note added: "Debug/Prg conn"
- note added: "Interface connector"
- note added: "RTC battery"
- note removed: "Debugger and programator connector"
- moved on the sheet: BT1, C1, C104, C105, D101, J103, J105, R102, R103, R108, SW102, U108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

Commit message: Final board schematics and sw setup
Parts:
- removed C105: 1u, Capacitor_SMD:C_0805_2012Metric_Pad1.18x1.45mm_HandSolder, symbol Device:C_Small
- removed C105: 100u, Capacitor_SMD:C_1210_3225Metric_Pad1.33x2.70mm_HandSolder, symbol Device:C_Small
- removed C107: 10u, Capacitor_SMD:C_0805_2012Metric_Pad1.18x1.45mm_HandSolder, symbol Device:C_Small
- removed C108: 100n, Capacitor_SMD:C_0805_2012Metric_Pad1.18x1.45mm_HandSolder, symbol Device:C_Small
- removed J105: DS1020-07-20VBT1B, Connector_FFC-FPC:TE_2-84952-0_1x20-1MP_P1.0mm_Horizontal, symbol Connector_Generic:Conn_01x20
- removed R108: 10k, Resistor_SMD:R_0805_2012Metric_Pad1.20x1.40mm_HandSolder, symbol Device:R_Small
- removed R108, R109, R110, R111: 3k3, Resistor_SMD:R_0805_2012Metric_Pad1.20x1.40mm_HandSolder, symbol Device:R_Small
- removed U1, U2, U3, U4: USBLC6-4SC6, Package_TO_SOT_SMD:SOT-23-6, symbol Power_Protection:USBLC6-4SC6
- removed U105: STM32G030C8T6, Package_QFP:LQFP-48_7x7mm_P0.5mm, symbol CustomSymbols:STM32G030C8T6
- removed U108: AP22802AW5-7, Package_TO_SOT_SMD:SOT-23-5, symbol Power_Management:AP22804AW5
- J103, J106: footprint Connector_PinHeader_2.54mm:PinHeader_2x03_P2.54mm_Vertical -> Connector_PinSocket_1.27mm:PinSocket_1x06_P1.27mm_Vertical_SMD_Pin1Left
- renumbered BT1 to BT101, C109 to C113, C1 to C116, J2 to J102, R4 to R108, R3 to R109, R1 to R110, R2 to R111, U110 to U104, U106 to U105, U104 to U106
Connections:
- net RF_DIO_2 is gone; now on net SPI1_MISO: U106.21 (PB2)
- net RF_DIO_3 is gone; now on net SPI2_SCK: U106.22 (PB10)
- net RF_DIO_4 is gone; now on net SPI2_MOSI: U106.23 (PB11)
- net GNDD: now also J103.5 (Pin_5), J106.5 (Pin_5)
- net SPI2_MISO: now also J103.2 (Pin_2); no longer J103.3 (Pin_3), U106.14 (PA3)
- net SPI2_MOSI: now also J103.3 (Pin_3); no longer J103.4 (Pin_4), U106.15 (PA4)
- net SPI2_SCK: now also J103.4 (Pin_4); no longer J103.5 (Pin_5), U106.11 (PA0)
- net ~{ERR_LED}: now also U106.37 (PA15); no longer U106.38 (PD0)
- net GPIO_A1 renamed GPIO_PA1
- net GPIO_PA1: no longer J103.1 (Pin_1)
- net GPIO_A2 renamed GPIO_PA2
- net GPIO_PA2: no longer J103.2 (Pin_2)
- net GPIO_A8 renamed GPIO_PA8
- net GPIO_B15 renamed GPIO_PB15
- net GPIO_PB15: no longer U106.37 (PA15)
- net GPIO_C6 renamed GPIO_PC6
- net GPIO_C7 renamed GPIO_PC7
- net GPIO_D1 renamed GPIO_PD1
- net GPIO_D2 renamed GPIO_PD2
- net GPIO_D3 renamed GPIO_PD3
- net RF_DIO_0 renamed RF_RESET
- net RF_DIO_1 renamed RF_FIFO_F_NE
- net RF_DIO_5 renamed SPI2_NSS
- net SPI2_NSS: now also J103.1 (Pin_1)
- new net GPIO_PA0: U106.11 (PA0)
- new net GPIO_PA3: U106.14 (PA3)
- new net GPIO_PA4: U106.15 (PA4)
- new net GPIO_PD0: U106.38 (PD0)
- no-connect marks 8 -> 11
Other:
- added sheet ExpansionConnector (ExpansionConnector.kicad_sch)
- note added: "Board expansion connectors"
- note removed: "ESD protection"
- note removed: "Interface connector"
- note removed: "ZAMIENIC NA G07"
- moved on the sheet: BT101, C104, C112, C113, C114, C115, C116, D101, J102, R102, R103, R108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

Commit message: layout dev
Parts:
- removed BT101: RTC_Bat, Battery:BatteryHolder_Keystone_3002_1x2032, symbol Device:Battery_Cell
- removed C104: 10u, Capacitor_SMD:C_0805_2012Metric_Pad1.18x1.45mm_HandSolder, symbol Device:C_Small
- removed C116: 100n, Capacitor_SMD:C_0805_2012Metric_Pad1.18x1.45mm_HandSolder, symbol Device:C_Small
- removed R102: 2k, Resistor_SMD:R_0805_2012Metric_Pad1.20x1.40mm_HandSolder, symbol Device:R_Small
- added H101, H102, H103, H104: MountingHole, MountingHole:MountingHole_3.2mm_M3, symbol Mechanical:MountingHole
- added U107: APX823, Package_TO_SOT_SMD:SOT-23-5_HandSoldering, symbol CustomSymbols:APX823-29W5G-7
- J102: footprint Connector_IDC:IDC-Header_2x10_P2.54mm_Horizontal -> Connector_IDC:IDC-Header_2x10_P2.54mm_Vertical_SMD
- R108, R109, R110, R111: footprint Resistor_SMD:R_0805_2012Metric_Pad1.20x1.40mm_HandSolder -> Resistor_SMD:R_0402_1005Metric_Pad0.72x0.64mm_HandSolder
- SW102: symbol Switch:SW_Push -> Switch:SW_MEC_5E
Connections:
- net +3V3: now also U107.5 (VCC)
- net GNDD: now also J106.3 (Pin_3), J106.4 (Pin_4), SW102.2, U107.2 (GND); no longer J106.5 (Pin_5), J106.6 (Pin_6)
- net I2C2_SCL_MEM: now also J106.6 (Pin_6); no longer J106.4 (Pin_4)
- net I2C2_SDA_MEM: now also J106.5 (Pin_5); no longer J106.3 (Pin_3)
- net SPI1_MISO: no longer U106.21 (PB2)
- net SPI2_MISO: now also U106.21 (PB2)
- net ~{RESET}: now also U107.1 (~{RESET}); no longer SW102.2
- new net: SW102.3 (K), SW102.4 (A), U107.3 (~{MR})
- no-connect marks 11 -> 12
Other:
- note added: "Error indicator LED"
- note added: "Mounting holes"
- note added: "PoR controler"
- note removed: "Error indicator LED and RESET button"
- note removed: "RTC battery"

Commit message: layout dev part 2
Parts:
- removed C101: 100n, Capacitor_SMD:C_0805_2012Metric_Pad1.18x1.45mm_HandSolder, symbol Device:C_Small
- removed C103: 1u, Capacitor_SMD:C_0805_2012Metric_Pad1.18x1.45mm_HandSolder, symbol Device:C_Small
- removed R104: 2k, Resistor_SMD:R_0402_1005Metric_Pad0.72x0.64mm_HandSolder, symbol Device:R_Small
- added C102: 100n, Capacitor_SMD:C_0402_1005Metric_Pad0.74x0.62mm_HandSolder, symbol Device:C_Small
- added C107: 4u7, Capacitor_SMD:C_0805_2012Metric_Pad1.18x1.45mm_HandSolder, symbol Device:C_Small
- added R103: 4k7, Resistor_SMD:R_0402_1005Metric_Pad0.72x0.64mm_HandSolder, symbol Device:R_Small
- added R104 (x2): 27, Resistor_SMD:R_0402_1005Metric_Pad0.72x0.64mm_HandSolder, symbol Device:R_Small
- added R113: 10k, Resistor_SMD:R_0402_1005Metric_Pad0.72x0.64mm_HandSolder, symbol Device:R_Small
Connections:
- net GPIO_B3 is gone; now on net GPIO_PB3: U106.42 (PB3)
- net GPIO_B4 is gone; now on net GPIO_PB4: U106.43 (PB4)
- net GPIO_B5 is gone; now on net GPIO_PB5: U106.44 (PB5)
- net GPIO_B8 is gone; now on net GPIO_PB8: U106.47 (PB8)
- net GPIO_B9 is gone; now on net GPIO_PB9: U106.48 (PB9)
- net +3V3: now also U102.10 (VCC), C107.1; no longer J102.1 (VTREF), J102.2 (VCC/NC), U102.8 (3V3OUT)
- net +5V: now also R103.1; no longer U102.10 (VCC)
- net GNDD: now also C102.2, C107.2, R113.2
- net I2C2_SCL_MEM: now also U106.33 (PA11/PA9); no longer U106.25 (PB13)
- net I2C2_SDA_MEM: now also U106.34 (PA12/PA10); no longer U106.26 (PB14)
- net USB_D+: now also R104.2; no longer U101.3 (I/O2)
- net USB_D-: now also R104.1; no longer U101.1 (I/O1)
- net at U102.9 (~{RESET}): now also U102.8 (3V3OUT), C102.1
- net at U102.12 (CBUS0): now also R103.2, R113.1
- net GPIO_C13 renamed GPIO_PC13
- net USART1_CTS: no longer names the net of U102.4 (~{CTS})
- net USART1_CTS: no longer U106.33 (PA11/PA9)
- net USART1_RTS: no longer names the net of U102.16 (~{RTS})
- net USART1_RTS: no longer U106.34 (PA12/PA10)
- new net CON_PWR: J102.1 (VTREF), J102.2 (VCC/NC)
- new net GPIO_PB13: U106.25 (PB13)
- new net GPIO_PB14: U106.26 (PB14)
- new net USB_RES+: R104.1, U101.3 (I/O2)
- new net USB_RES-: R104.2, U101.1 (I/O1)
- no-connect marks 12 -> 13
Other:
- sheet ExpansionConnector ports: added CON_PWR, GPIO_PB13, GPIO_PB14; removed none
- moved on the sheet: C102, U102

Commit message: Finished Giskard layout
- Need to fix DRC violations
- It'd be nice to move EEPROM closer to MPU
Parts:
- removed J106: Test pins COMM2, Connector_PinSocket_1.27mm:PinSocket_1x06_P1.27mm_Vertical_SMD_Pin1Left, symbol Connector_Generic:Conn_01x06
- added D101: PWR_LED, Diode_SMD:D_0805_2012Metric_Pad1.15x1.40mm_HandSolder, symbol Device:LED
- added R103: 330, Resistor_SMD:R_0805_2012Metric_Pad1.20x1.40mm_HandSolder, symbol Device:R_Small
- R103, R105, R106: value 270 -> 330
Connections:
- net GPIO_PB8 is gone; now on net I2C1_SCL: U106.47 (PB8)
- net GPIO_PB9 is gone; now on net I2C1_SDA: U106.48 (PB9)
- net GPIO_PD0 is gone; now on net SPI2_NSS: U106.38 (PD0)
- net GPIO_PD1 is gone; now on net SPI2_SCK: U106.39 (PD1)
- net GPIO_PD2 is gone; now on net RF_FIFO_F_NE: U106.40 (PD2)
- net GPIO_PD3 is gone; now on net RF_RESET: U106.41 (PD3)
- net +3V3: now also R103.1
- net GNDD: now also D101.1 (K)
- net I2C1_SCL: no longer U106.29 (PA9/NC)
- net I2C1_SDA: no longer U106.32 (PA10/NC)
- net RF_FIFO_F_NE: no longer U106.20 (PB1)
- net RF_RESET: no longer U106.19 (PB0)
- net SPI2_MISO: now also U106.45 (PB6); no longer U106.21 (PB2)
- net SPI2_MOSI: now also U106.46 (PB7); no longer U106.23 (PB11)
- net SPI2_NSS: no longer U106.24 (PB12)
- net SPI2_SCK: no longer U106.22 (PB10)
- net USART1_RX: now also U106.32 (PA10/NC); no longer U106.46 (PB7)
- net USART1_TX: now also U106.29 (PA9/NC); no longer U106.45 (PB6)
- new net: D101.2 (A), R103.2
- new net GPIO_PB0: U106.19 (PB0)
- new net GPIO_PB1: U106.20 (PB1)
- new net GPIO_PB10: U106.22 (PB10)
- new net GPIO_PB11: U106.23 (PB11)
- new net GPIO_PB12: U106.24 (PB12)
- new net GPIO_PB2: U106.21 (PB2)
Other:
- sheet ExpansionConnector ports: added GPIO_PB0, GPIO_PB1, GPIO_PB10, GPIO_PB11, GPIO_PB12, GPIO_PB2; removed GPIO_PB8, GPIO_PB9, GPIO_PD0, GPIO_PD1, GPIO_PD2, GPIO_PD3
- moved on the sheet: J101, J103, R104, U101

Commit message: Finished board layout
Parts:
- D101: value ERR_LED (RED) -> ERR_LED
Changed lines of the file:
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@@
   )
   (text "The _S suffix is\nfor \"Safe\" \n(from ESD threats :))"
-    (at 82.55 0.635 0)
+    (at 75.565 22.225 0)
     (effects (font (size 1.27 1.27)) (justify left bottom))
   )
@@
       (effects (font (size 1.27 1.27)) (justify right))
     )
-    (property "Value" "ERR_LED (RED)" (at 205.105 42.545 0)
-      (effects (font (size 1.27 1.27)) (justify right))
-    )
+    (property "Value" "ERR_LED" (at 205.105 42.545 0)
+      (effects (font (size 1.27 1.27)) (justify right))
+    )
