File: Hardware/Giskard_rev1/GiskardRF/RadioComm.kicad_sch (KiCad schematic)
At the start: 14 parts, among them J401 SMA6252A23G50, U402 RFM69HW

Commit message: Final board schematics and sw setup
Parts:
- J401: footprint Connector_Coaxial:SMA_Amphenol_901-143_Horizontal -> Connector_Coaxial:SMA_Samtec_SMA-J-P-X-ST-EM1_EdgeMount
Changed lines of the file:
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@@
       (effects (font (size 1.27 1.27)) (justify left))
     )
-    (property "Footprint" "Connector_Coaxial:SMA_Amphenol_901-143_Horizontal" (at 197.485 90.805 0)
+    (property "Footprint" "Connector_Coaxial:SMA_Samtec_SMA-J-P-X-ST-EM1_EdgeMount" (at 197.485 90.805 0)
       (effects (font (size 1.27 1.27)) hide)
     )

Commit message: layout dev
Connections:
- net SPI1_MISO: now also R402.2
- net SPI1_MOSI: no longer R402.2
Changed lines of the file:
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@@
   (junction (at 113.665 78.74) (diameter 0) (color 0 0 0 0)
   )
-  (junction (at 102.235 95.885) (diameter 0) (color 0 0 0 0)
+  (junction (at 102.235 93.345) (diameter 0) (color 0 0 0 0)
   )
   (junction (at 166.37 118.745) (diameter 0) (color 0 0 0 0)
@@
     (stroke (width 0) (type default))
   )
-  (wire (pts (xy 102.235 95.885) (xy 107.95 95.885))
+  (wire (pts (xy 90.805 95.885) (xy 107.95 95.885))
     (stroke (width 0) (type default))
   )
@@
     (stroke (width 0) (type default))
   )
-  (wire (pts (xy 90.805 95.885) (xy 102.235 95.885))
-    (stroke (width 0) (type default))
-  )
   (wire (pts (xy 181.61 121.285) (xy 181.61 118.745))
     (stroke (width 0) (type default))
@@
     (stroke (width 0) (type default))
   )
-  (wire (pts (xy 90.805 93.345) (xy 118.11 93.345))
+  (wire (pts (xy 90.805 93.345) (xy 102.235 93.345))
     (stroke (width 0) (type default))
   )
@@
     (stroke (width 0) (type default))
   )
+  (wire (pts (xy 102.235 93.345) (xy 118.11 93.345))
+    (stroke (width 0) (type default))
+  )
   (wire (pts (xy 172.72 118.745) (xy 172.72 115.57))
     (stroke (width 0) (type default))
@@
     (stroke (width 0) (type default))
   )
-  (wire (pts (xy 102.235 86.995) (xy 102.235 95.885))
+  (wire (pts (xy 102.235 86.995) (xy 102.235 93.345))
     (stroke (width 0) (type default))
   )
