File: Hardware/Giskard_rev1/GiskardRF/GiskardRF.kicad_pcb (KiCad board)
At the start: 4 copper layers, 64 parts, among them J101 USB_B_Micro, J102 DebugConn, J103 Test pins COMM1, J104 Test pins COMM2, J105 ExtensionConn, J201 SMA6252A23G50, SW101 RESET, U101 USBLC6-2P6, U102 FT230XQ, U103 AP22802AW5-7, U105 STM32G030C8T6, U106 M24C16-RM, U107 23K256-I/SN, U108 AP22802AW5-7, U110 AP2127K-3.3, U201 RFM69HW, Y101 3225-16M-SR 16MHz 9pF, Y102 32.768K-CFPX217

Commit message: Upgrade to stmg07
Parts:
- Y102: footprint Crystal:Crystal_SMD_TXC_7A-2Pin_5x3.2mm -> Crystal:Crystal_SMD_MicroCrystal_CC7V-T1A-2Pin_3.2x1.5mm_HandSoldering
- moved Y102 0.51 mm to (147.3, 135.6)
Routing:
- net /LF_OSC_OUT: track 7.25 -> 6.64 mm
- net /LF_OSC_IN: track 7.86 -> 7.26 mm
Changed lines of the file:
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@@
     )
   )
-  (footprint "Crystal:Crystal_SMD_TXC_7A-2Pin_5x3.2mm" (layer "F.Cu")
-    (at 147.3145 135.128)
-    (descr "SMD Crystal TXC 7A http://txccrystal.com/images/pdf/7a.pdf")
-    (tags "SMD SMT crystal")
+  (footprint "Crystal:Crystal_SMD_MicroCrystal_CC7V-T1A-2Pin_3.2x1.5mm_HandSoldering" (layer "F.Cu")
+    (at 147.3145 135.636)
+    (descr "SMD Crystal MicroCrystal CC7V-T1A/CM7V-T1A series http://www.microcrystal.com/images/_Product-Documentation/01_TF_ceramic_Packages/01_Datasheet/CC1V-T1A.pdf, hand-soldering, 3.2x1.5mm^2 package")
+    (tags "SMD SMT crystal hand-soldering")
     (property "Sheetfile" "GiskardRF.kicad_sch")
     (property "Sheetname" "")
@@
     (property "ki_keywords" "quartz ceramic resonator oscillator")
     (attr smd)
-    (fp_text reference "Y102" (at -0.254 -2.794) (layer "F.SilkS")
-        (effects (font (size 1 1) (thickness 0.15)))
-    )
-    (fp_text value "32.768K-CFPX217" (at 0 2.7) (layer "F.Fab") hide
-        (effects (font (size 1 1) (thickness 0.15)))
-    )
-    (fp_text user "${REFERENCE}" (at 0.072 0) (layer "F.Fab")
-        (effects (font (size 1 1) (thickness 0.15)))
-    )
-    (fp_line (start -2.5 -1.71) (end 2.5 -1.71)
-      (stroke (width 0.12) (type solid)) (layer "F.SilkS"))
-    (fp_line (start -2.5 1.71) (end 2.5 1.71)
-      (stroke (width 0.12) (type solid)) (layer "F.SilkS"))
-    (fp_line (start -2.95 -1.85) (end -2.95 1.85)
-      (stroke (width 0.05) (type solid)) (layer "F.CrtYd"))
-    (fp_line (start -2.95 -1.85) (end 2.95 -1.85)
-      (stroke (width 0.05) (type solid)) (layer "F.CrtYd"))
-    (fp_line (start 2.95 -1.85) (end 2.95 1.85)
-      (stroke (width 0.05) (type solid)) (layer "F.CrtYd"))
-    (fp_line (start 2.95 1.85) (end -2.95 1.85)
-      (stroke (width 0.05) (type solid)) (layer "F.CrtYd"))
-    (fp_line (start -2.5 -1.6) (end -2.5 1.6)
-      (stroke (width 0.1) (type solid)) (layer "F.Fab"))
-    (fp_line (start -2.5 -1.6) (end 2.5 -1.6)
-      (stroke (width 0.1) (type solid)) (layer "F.Fab"))
-    (fp_line (start -2.5 1.6) (end 2.5 1.6)
-      (stroke (width 0.1) (type solid)) (layer "F.Fab"))
-    (fp_line (start 2.5 -1.6) (end 2.5 1.6)
-      (stroke (width 0.1) (type solid)) (layer "F.Fab"))
-    (pad "1" smd rect (at -1.85 0) (size 1.7 2.4) (layers "F.Cu" "F.Paste" "F.Mask")
+    (fp_text reference "Y102" (at 0 -1.95) (layer "F.SilkS")
+        (effects (font (size 1 1) (thickness 0.15)))
+    )
+    (fp_text value "32.768K-CFPX217" (at 0 1.95) (layer "F.Fab") hide
+        (effects (font (size 1 1) (thickness 0.15)))
+    )
+    (fp_text user "${REFERENCE}" (at 0 0) (layer "F.Fab")
+        (effects (font (size 0.7 0.7) (thickness 0.105)))
+    )
+    (fp_line (start -2.7 -0.9) (end -2.7 0.9)
+      (stroke (width 0.12) (type solid)) (layer "F.SilkS"))
+    (fp_line (start -0.55 -0.95) (end 0.55 -0.95)
+      (stroke (width 0.12) (type solid)) (layer "F.SilkS"))
+    (fp_line (start -0.55 0.95) (end 0.55 0.95)
+      (stroke (width 0.12) (type solid)) (layer "F.SilkS"))
+    (fp_line (start -2.8 -1.2) (end -2.8 1.2)
+      (stroke (width 0.05) (type solid)) (layer "F.CrtYd"))
+    (fp_line (start -2.8 1.2) (end 2.8 1.2)
+      (stroke (width 0.05) (type solid)) (layer "F.CrtYd"))
+    (fp_line (start 2.8 -1.2) (end -2.8 -1.2)
+      (stroke (width 0.05) (type solid)) (layer "F.CrtYd"))
+    (fp_line (start 2.8 1.2) (end 2.8 -1.2)
+      (stroke (width 0.05) (type solid)) (layer "F.CrtYd"))
+    (fp_line (start -1.6 -0.75) (end -1.6 0.75)
+      (stroke (width 0.1) (type solid)) (layer "F.Fab"))
+    (fp_line (start -1.6 0.25) (end -1.1 0.75)
+      (stroke (width 0.1) (type solid)) (layer "F.Fab"))
+    (fp_line (start -1.6 0.75) (end 1.6 0.75)
+      (stroke (width 0.1) (type solid)) (layer "F.Fab"))
+    (fp_line (start 1.6 -0.75) (end -1.6 -0.75)
+      (stroke (width 0.1) (type solid)) (layer "F.Fab"))
+    (fp_line (start 1.6 0.75) (end 1.6 -0.75)
+      (stroke (width 0.1) (type solid)) (layer "F.Fab"))
+    (pad "1" smd rect (at -1.625 0) (size 1.75 1.8) (layers "F.Cu" "F.Paste" "F.Mask")
       (net 7 "/LF_OSC_OUT") (pinfunction "1") (pintype "passive"))
-    (pad "2" smd rect (at 1.85 0) (size 1.7 2.4) (layers "F.Cu" "F.Paste" "F.Mask")
+    (pad "2" smd rect (at 1.625 0) (size 1.75 1.8) (layers "F.Cu" "F.Paste" "F.Mask")
       (net 6 "/LF_OSC_IN") (pinfunction "2") (pintype "passive"))
-    (model "${KICAD6_3DMODEL_DIR}/Crystal.3dshapes/Crystal_SMD_TXC_7A-2Pin_5x3.2mm.wrl"
+    (model "${KICAD6_3DMODEL_DIR}/Crystal.3dshapes/Crystal_SMD_MicroCrystal_CC7V-T1A-2Pin_3.2x1.5mm_HandSoldering.wrl"
       (offset (xyz 0 0 0))
       (scale (xyz 1 1 1))
@@
   (segment (start 105.654 141.996) (end 105.918 141.732) (width 0.3) (layer "F.Cu") (net 5))
   (segment (start 104.3 141.996) (end 105.654 141.996) (width 0.3) (layer "F.Cu") (net 5))
-  (segment (start 149.1645 135.128) (end 148.3305 135.962) (width 0.3) (layer "F.Cu") (net 6))
+  (segment (start 148.3305 136.245) (end 148.9395 135.636) (width 0.3) (layer "F.Cu") (net 6))
   (segment (start 148.0765 137.922) (end 147.3145 137.922) (width 0.3) (layer "F.Cu") (net 6))
-  (segment (start 148.3305 135.962) (end 148.3305 137.668) (width 0.3) (layer "F.Cu") (net 6))
   (segment (start 147.3145 137.922) (end 145.7905 139.446) (width 0.3) (layer "F.Cu") (net 6))
   (segment (start 148.3305 137.668) (end 148.0765 137.922) (width 0.3) (layer "F.Cu") (net 6))
+  (segment (start 148.3305 137.668) (end 148.3305 136.245) (width 0.3) (layer "F.Cu") (net 6))
   (segment (start 145.7905 139.82002) (end 146.724158 140.753678) (width 0.3) (layer "F.Cu") (net 6))
   (segment (start 145.7905 139.446) (end 145.7905 139.82002) (width 0.3) (layer "F.Cu") (net 6))
-  (segment (start 146.358 136.0215) (end 146.358 137.668) (width 0.3) (layer "F.Cu") (net 7))
   (segment (start 145.2825 140.019126) (end 146.370605 141.107231) (width 0.3) (layer "F.Cu") (net 7))
-  (segment (start 145.4645 135.128) (end 146.358 136.0215) (width 0.3) (layer "F.Cu") (net 7))
+  (segment (start 146.358 136.3045) (end 145.6895 135.636) (width 0.3) (layer "F.Cu") (net 7))
   (segment (start 145.2825 139.192) (end 145.2825 140.019126) (width 0.3) (layer "F.Cu") (net 7))
   (segment (start 146.358 138.1165) (end 145.2825 139.192) (width 0.3) (layer "F.Cu") (net 7))
   (segment (start 146.358 137.668) (end 146.358 138.1165) (width 0.3) (layer "F.Cu") (net 7))
+  (segment (start 146.358 137.668) (end 146.358 136.3045) (width 0.3) (layer "F.Cu") (net 7))
   (segment (start 140.511362 140.11861) (end 141.139344 140.11861) (width 0.3) (layer "F.Cu") (net 8))
   (segment (start 141.139344 140.11861) (end 144.249285 143.228551) (width 0.3) (layer "F.Cu") (net 8))

Commit message: Final board schematics and sw setup
Parts:
- removed C117: 1u, Capacitor_SMD:C_0805_2012Metric_Pad1.18x1.45mm_HandSolder
- removed C118: 100u, Capacitor_SMD:C_1210_3225Metric_Pad1.33x2.70mm_HandSolder
- removed J105: ExtensionConn, Connector_IDC:IDC-Header_2x10_P2.54mm_Horizontal
- removed R112: 1k, Resistor_SMD:R_0805_2012Metric_Pad1.20x1.40mm_HandSolder
- removed R113: 10k, Resistor_SMD:R_0805_2012Metric_Pad1.20x1.40mm_HandSolder
- removed the U105 at (148.1, 145.3)
- removed U107: 23K256-I/SN, Package_SO:SO-8_3.9x4.9mm_P1.27mm
- removed U108: AP22802AW5-7, Package_TO_SOT_SMD:SOT-23-5
- added BT101: RTC_Bat, Battery:BatteryHolder_Keystone_3002_1x2032, F.Cu at (106.8, 60.2)
- added C301: 1u, Capacitor_SMD:C_0805_2012Metric_Pad1.18x1.45mm_HandSolder, F.Cu at (95.6, 105.7)
- added C302: 100u, Capacitor_SMD:C_1210_3225Metric_Pad1.33x2.70mm_HandSolder, F.Cu at (96.2, 102.1)
- added J301: Conn_02x05_Odd_Even, Connector_PinHeader_1.27mm:PinHeader_2x05_P1.27mm_Vertical_SMD, F.Cu at (96.1, 87.9)
- added J302: Conn_02x05_Odd_Even, Connector_PinHeader_1.27mm:PinHeader_2x05_P1.27mm_Vertical_SMD, F.Cu at (88.4, 90.5)
- added J303: Conn_02x05_Odd_Even, Connector_PinHeader_1.27mm:PinHeader_2x05_P1.27mm_Vertical_SMD, F.Cu at (88.4, 98.9)
- added J304: Conn_02x05_Odd_Even, Connector_PinHeader_1.27mm:PinHeader_2x05_P1.27mm_Vertical_SMD, F.Cu at (96.1, 94.7)
- added R301: 10k, Resistor_SMD:R_0805_2012Metric_Pad1.20x1.40mm_HandSolder, F.Cu at (85.9, 104.6)
- added U106: STM32G070CBTx, Package_QFP:LQFP-48_7x7mm_P0.5mm, F.Cu at (158.7, 123.4)
- added U301: USBLC6-4SC6, Package_TO_SOT_SMD:SOT-23-6, F.Cu at (75.8, 88.5)
- added U302: USBLC6-4SC6, Package_TO_SOT_SMD:SOT-23-6, F.Cu at (75.8, 92.9)
- added U303: AP22802AW5-7, Package_TO_SOT_SMD:SOT-23-5, F.Cu at (75.8, 97.4)
- added U304: USBLC6-4SC6, Package_TO_SOT_SMD:SOT-23-6, F.Cu at (75.8, 101.8)
- added U305: USBLC6-4SC6, Package_TO_SOT_SMD:SOT-23-6, F.Cu at (75.8, 106.3)
- added U306: USBLC6-4SC6, Package_TO_SOT_SMD:SOT-23-6, F.Cu at (81.0, 88.5)
- added U308: USBLC6-4SC6, Package_TO_SOT_SMD:SOT-23-6, F.Cu at (81.0, 97.4)
- C109: renamed from C110; value 100n -> 20p
- C110: renamed from C111; value 100n -> 20p
- C111: renamed from C112; value 100n -> 13p
- C112: renamed from C113; value 100n -> 13p
- C114, C115: moved to F.Cu
- J102: value DebugConn -> Conn_ARM_JTAG_SWD_20; footprint Connector_IDC:IDC-Header_2x03_P2.54mm_Vertical -> Connector_IDC:IDC-Header_2x10_P2.54mm_Horizontal
- J103: renamed from J104; footprint Connector_PinHeader_2.54mm:PinHeader_2x03_P2.54mm_Vertical -> Connector_PinSocket_1.27mm:PinSocket_1x06_P1.27mm_Vertical_SMD_Pin1Left
- J104: renamed from J103; footprint Connector_PinHeader_2.54mm:PinHeader_2x03_P2.54mm_Vertical -> Connector_PinSocket_1.27mm:PinSocket_1x06_P1.27mm_Vertical_SMD_Pin1Left
- J201: footprint Connector_Coaxial:SMA_Amphenol_901-143_Horizontal -> Connector_Coaxial:SMA_Samtec_SMA-J-P-X-ST-EM1_EdgeMount
- moved J102 83.5 mm to (76.2, 55.3), turned to 0 degrees
- moved C114 77.6 mm to (109.0, 73.3), turned to 0 degrees
- moved R111 77.6 mm to (92.8, 82.1)
- moved C115 72.8 mm to (109.0, 76.3), turned to 0 degrees
- moved R108 68.7 mm to (92.8, 73.3)
- moved R109 68.7 mm to (92.8, 76.2)
- moved R110 68.7 mm to (92.8, 79.2)
- moved C116 46.2 mm to (109.0, 79.3)
- moved J103 13.3 mm to (106.3, 168.3)
- renumbered C109 to C113, U110 to U104, U106 to U105
Connections:
- net /RF_DIO_0 renamed /RadioComm1/RF_DIO0
- net /RF_DIO_1 renamed /RF_FIFO_F_NE
- net /RF_DIO_2 renamed /RadioComm1/RF_DIO2
- net /RF_DIO_3 renamed /RadioComm1/RF_DIO3
- net /RF_DIO_4 renamed /RadioComm1/RF_DIO4
- net /RF_DIO_5 renamed /RadioComm1/RF_DIO5
- net /RadioComm1/RF_RESET renamed /RF_RESET
- C116 pad 1: +3V3 -> /3V_Bat
- J102 pad 3: /SW_CLK -> GNDD
- J102 pad 4: /SW_DIO -> GNDD
- J103 pad 3: /USART1_RTS -> /I2C2_SDA_MEM
- J103 pad 4: /USART1_CTS -> /I2C2_SCL_MEM
- J103 pad 5: unconnected-(J104-Pin_5-Pad5) -> GNDD
- J104 pad 1: /GPIO_A1 -> /SPI2_NSS
- J104 pad 2: /GPIO_A2 -> /SPI2_MISO
- J104 pad 3: /SPI1_MOSI -> /SPI2_MOSI
- J104 pad 4: /SPI1_MISO -> /SPI2_SCK
- J104 pad 5: /SPI1_SCK -> GNDD
- R108 pad 2: /I2C2_SCL_MEM -> /I2C2_SDA_MEM
- R204 pad 2: /GPIO_A2 -> /GPIO_PB11
- U201 pad 15: /GPIO_A2 -> /GPIO_PB11

Commit message: layout dev
Parts:
- removed BT101: RTC_Bat, Battery:BatteryHolder_Keystone_3002_1x2032
- removed C104: 10u, Capacitor_SMD:C_0805_2012Metric_Pad1.18x1.45mm_HandSolder
- removed C116: 100n, Capacitor_SMD:C_0805_2012Metric_Pad1.18x1.45mm_HandSolder
- removed R101: 2k, Resistor_SMD:R_0805_2012Metric_Pad1.20x1.40mm_HandSolder
- added H101: MountingHole, MountingHole:MountingHole_3.2mm_M3, F.Cu at (188.7, 136.1)
- added H102: MountingHole, MountingHole:MountingHole_3.2mm_M3, F.Cu at (116.1, 136.1)
- added H103: MountingHole, MountingHole:MountingHole_3.2mm_M3, F.Cu at (116.1, 99.6)
- added H104: MountingHole, MountingHole:MountingHole_3.2mm_M3, F.Cu at (188.7, 99.6)
- added U107: APX823, Package_TO_SOT_SMD:SOT-23-5_HandSoldering, F.Cu at (162.5, 111.8)
- C114, C115, C201, C301, C302, J301, J302, J303, J304, R201, R202, R203, R204, R205, R206, R207, R208, R209, R210, R211, R301, U301, U302, U303, U304, U305, U306, U308: moved to B.Cu
- J102: footprint Connector_IDC:IDC-Header_2x10_P2.54mm_Horizontal -> Connector_IDC:IDC-Header_2x10_P2.54mm_Vertical_SMD
- R108, R109, R110, R111: footprint Resistor_SMD:R_0805_2012Metric_Pad1.20x1.40mm_HandSolder -> Resistor_SMD:R_0402_1005Metric_Pad0.72x0.64mm_HandSolder
- moved J102 107.3 mm to (151.6, 131.6), turned to -90 degrees
- moved U302 105.2 mm to (172.3, 134.7), turned to 180 degrees
- moved U305 95.4 mm to (171.1, 101.7), turned to 90 degrees
- moved SW101 92.1 mm to (128.5, 133.6), turned to 180 degrees
- moved U303 84.5 mm to (153.4, 130.7)
- moved J303 83.9 mm to (164.6, 133.9), turned to -90 degrees
- moved U105 82.9 mm to (148.8, 100.4), turned to 0 degrees
- moved J103 79.7 mm to (177.2, 131.9), turned to 90 degrees
- moved U306 78.1 mm to (157.9, 101.7), turned to 90 degrees
- moved J201 77.3 mm to (179.3, 98.1), turned to 180 degrees
- moved R301 75.7 mm to (155.7, 133.9), turned to 180 degrees
- moved R110 72.6 mm to (162.2, 100.7)
- moved U301 71.7 mm to (131.6, 133.6), turned to 180 degrees
- moved R111 71.1 mm to (159.6, 106.7)
- moved J302 70.5 mm to (144.0, 133.8), turned to -90 degrees
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Connections:
- J103 pad 3: /I2C2_SDA_MEM -> GNDD
- J103 pad 4: /I2C2_SCL_MEM -> GNDD
- J103 pad 5: GNDD -> /I2C2_SDA_MEM
- J103 pad 6: GNDD -> /I2C2_SCL_MEM
- J301 pad 2: /ExpansionConnector/CONTACT_PWR -> GNDD
- J302 pad 2: /ExpansionConnector/CONTACT_PWR -> GNDD
- J303 pad 4: GNDD -> /ExpansionConnector/CONTACT_PWR
- J303 pad 6: GNDD -> /ExpansionConnector/CONTACT_PWR
- J304 pad 2: /ExpansionConnector/CONTACT_PWR -> GNDD
- R202 pad 2: /SPI2_MOSI -> /SPI2_MISO
- SW101 pad 2: /~{RESET} -> GNDD
- U106 pad 21: /SPI1_MISO -> /SPI2_MISO
Routing:
- net GNDD: track 49.5 -> 115.7 mm, vias 13 -> 24
- net +3V3: track 64.8 -> 78.9 mm, vias 3 -> 10
- net /I2C2_SDA_MEM: track 0.00 -> 7.84 mm
- net /RF_RESET: track 0.00 -> 5.73 mm, vias 0 -> 1
- net /~{RESET}: track 0.00 -> 5.67 mm
- net /RadioComm1/RF_DIO0: track 0.00 -> 5.63 mm, vias 0 -> 1
- net /RF_FIFO_F_NE: track 0.00 -> 5.48 mm, vias 0 -> 1
- net /RadioComm1/RF_DIO2: track 0.00 -> 5.39 mm, vias 0 -> 1
- net /I2C2_SCL_MEM: track 0.00 -> 5.34 mm
- net /RadioComm1/RF_DIO3: track 0.00 -> 5.29 mm, vias 0 -> 1
- net /RadioComm1/RF_DIO4: track 0.00 -> 5.19 mm, vias 0 -> 1
- net /RadioComm1/RF_DIO5: track 0.00 -> 5.10 mm, vias 0 -> 1
- net /~{ERR_LED}: track 0.00 -> 2.52 mm
- net Net-(D101-A): track 0.00 -> 2.27 mm
- net /HF_OSC_OUT: track 5.03 -> 6.65 mm
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- added copper zone on In2.Cu, net +3V3
- added copper zone on In1.Cu, net GNDD
Other:
- board outline added: 79.8 x 43.7 mm

Commit message: layout dev part 2
Parts:
- removed C103: 1u, Capacitor_SMD:C_0805_2012Metric_Pad1.18x1.45mm_HandSolder
- removed U301, U302, U304, U305, U306, U308: USBLC6-4SC6, Package_TO_SOT_SMD:SOT-23-6
- added C104: 100n, Capacitor_SMD:C_0402_1005Metric_Pad0.74x0.62mm_HandSolder, F.Cu at (107.4, 120.7)
- added R101: 27, Resistor_SMD:R_0402_1005Metric_Pad0.72x0.64mm_HandSolder, F.Cu at (120.9, 109.5)
- added R112: 27, Resistor_SMD:R_0402_1005Metric_Pad0.72x0.64mm_HandSolder, F.Cu at (120.9, 108.2)
- added R113: 10k, Resistor_SMD:R_0402_1005Metric_Pad0.72x0.64mm_HandSolder, F.Cu at (104.2, 122.7)
- C101: value 100n -> 4u7
- R103: value 2k -> 4k7
- moved J303 41.2 mm to (139.7, 101.1)
- moved J301 39.8 mm to (167.9, 133.6), turned to 90 degrees
- moved C114 39.8 mm to (190.0, 91.9)
- moved C115 39.8 mm to (190.0, 88.4)
- moved J304 39.6 mm to (138.2, 131.2), turned to -90 degrees
- moved J302 38.4 mm to (164.1, 101.1), turned to 90 degrees
- moved R111 28.1 mm to (148.3, 81.0)
- moved R103 19.8 mm to (104.2, 120.7), turned to 0 degrees
- moved R110 17.5 mm to (171.4, 85.9)
- moved C101 15.4 mm to (104.9, 118.2), turned to 0 degrees
- moved U101 2.99 mm to (125.9, 108.9)
- moved C102 2.65 mm to (122.2, 113.0), turned to -90 degrees
- moved R104 1.61 mm to (117.7, 122.1)
- moved R105 1.61 mm to (121.2, 122.1)
- moved D102 1.61 mm to (117.7, 118.0)
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Connections:
- C101 pad 1: +5V -> +3V3
- C301 pad 1: /ExpansionConnector/CONTACT_PWR -> /CON_PWR
- J102 pad 1: +3V3 -> /CON_PWR
- J102 pad 2: +3V3 -> /CON_PWR
- J301 pad 1: /GPIO_PB8 -> /GPIO_PD3
- J301 pad 10: /GPIO_C13 -> /GPIO_PB4
- J301 pad 2: GNDD -> /GPIO_PC13
- J301 pad 3: /GPIO_PB9 -> GNDD
- J301 pad 4: GNDD -> /GPIO_PB9
- J301 pad 6: /GPIO_PC6 -> /GPIO_PB8
- J301 pad 8: /GPIO_PC7 -> /GPIO_PB5
- J301 pad 9: GNDD -> /GPIO_PB3
- J302 pad 1: /I2C1_SCL -> /GPIO_PA3
- J302 pad 10: /SPI1_MOSI -> GNDD
- J302 pad 2: GNDD -> /GPIO_PA2
- J302 pad 3: /I2C1_SDA -> /GPIO_PA4
- J302 pad 4: GNDD -> /GPIO_PA1
- J302 pad 5: GNDD -> /SPI1_SCK
- J302 pad 6: /GPIO_PA4 -> GNDD
- J302 pad 7: /SPI1_SCK -> /SPI1_MISO
- J302 pad 9: /SPI1_MISO -> /SPI1_MOSI
- J303 pad 1: /GPIO_PA0 -> GNDD
- J303 pad 10: /GPIO_PB15 -> /GPIO_PA8
- J303 pad 2: /ExpansionConnector/CONTACT_PWR -> /CON_PWR
- J303 pad 3: /GPIO_PA1 -> GNDD
- J303 pad 4: /ExpansionConnector/CONTACT_PWR -> /CON_PWR
- J303 pad 5: GNDD -> /GPIO_PA0
- J303 pad 6: /ExpansionConnector/CONTACT_PWR -> /CON_PWR
- J303 pad 7: /GPIO_PA2 -> /GPIO_PB13
- J303 pad 8: /GPIO_PA8 -> /GPIO_PB15
- J303 pad 9: /GPIO_PA3 -> /GPIO_PB14
- J304 pad 10: /GPIO_PB4 -> /I2C1_SDA
- J304 pad 2: GNDD -> /I2C1_SCL
- J304 pad 7: /GPIO_PD3 -> /GPIO_PC7
- J304 pad 8: /GPIO_PB5 -> GNDD
- J304 pad 9: /GPIO_PB3 -> /GPIO_PC6
- R103 pad 1: +3V3 -> +5V
- R103 pad 2: Net-(U102-~{RESET}) -> Net-(U102-CBUS0)
- R204 pad 2: /GPIO_PB11 -> /SPI2_NSS
- R301 pad 1: /ExpansionConnector/CONTACT_PWR -> /CON_PWR
- U101 pad 1: /USB_D- -> /USB_RES-
- U101 pad 3: /USB_D+ -> /USB_RES+
- U102 pad 10: +5V -> +3V3
- U102 pad 12: unconnected-(U102-CBUS0-Pad12) -> Net-(U102-CBUS0)
- U102 pad 16: /USART1_RTS -> unconnected-(U102-~{RTS}-Pad16)
- U102 pad 4: /USART1_CTS -> unconnected-(U102-~{CTS}-Pad4)
- U102 pad 8: +3V3 -> Net-(U102-3V3OUT)
- U102 pad 9: Net-(U102-~{RESET}) -> Net-(U102-3V3OUT)
- U106 pad 1: /GPIO_C13 -> /GPIO_PC13
- U106 pad 25: /I2C2_SCL_MEM -> /GPIO_PB13
- U106 pad 26: /I2C2_SDA_MEM -> /GPIO_PB14
- U106 pad 33: /USART1_CTS -> /I2C2_SCL_MEM
- U106 pad 34: /USART1_RTS -> /I2C2_SDA_MEM
- U106 pad 42: /GPIO_B3 -> /GPIO_PB3
- U106 pad 43: /GPIO_B4 -> /GPIO_PB4
- U106 pad 44: /GPIO_B5 -> /GPIO_PB5
- U106 pad 47: /GPIO_B8 -> /GPIO_PB8
- U106 pad 48: /GPIO_B9 -> /GPIO_PB9
- U201 pad 15: /GPIO_PB11 -> /SPI2_NSS
- U303 pad 5: /ExpansionConnector/CONTACT_PWR -> /CON_PWR
Routing:
- net +3V3: track 78.9 -> 38.7 mm
- net +5V: track 38.1 -> 18.3 mm, vias 2 -> 0
- net GNDD: track 115.7 -> 100.6 mm, vias 24 -> 22
- net /USB_D-: track 11.5 -> 3.79 mm
- net /USB_D+: track 11.4 -> 3.75 mm
- net /USART1_CTS: track 6.56 -> 0.00 mm, vias 2 -> 0
- net /USB_D_S+: track 7.31 -> 1.62 mm
- net /USB_RES+: track 0.00 -> 3.83 mm
- net /USB_RES-: track 0.00 -> 3.82 mm
- net /I2C2_SDA_MEM: track 7.84 -> 4.05 mm
- net /I2C2_SCL_MEM: track 5.34 -> 1.70 mm
- net /USART1_TX: track 4.46 -> 1.32 mm, vias 2 -> 0
- net /USB_D_S-: track 7.37 -> 4.36 mm
- net Net-(U102-~{RESET}): track 1.70 -> 0.00 mm
- net /5V_USB: track 30.7 -> 29.4 mm
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
Commit message: Layout dev part 3
Parts:
- removed J301, J302, J303, J304: Conn_02x05_Odd_Even, Connector_PinHeader_1.27mm:PinHeader_2x05_P1.27mm_Vertical_SMD
- added J305: Conn_01x16, Connector_PinHeader_2.54mm:PinHeader_1x16_P2.54mm_Vertical_SMD_Pin1Left, B.Cu at (144.3, 100.7)
- added J306: Conn_01x16, Connector_PinHeader_2.54mm:PinHeader_1x16_P2.54mm_Vertical_SMD_Pin1Left, B.Cu at (144.5, 135.0)
- C102, C104, R103, R113, U102: moved to B.Cu
- moved C115 49.5 mm to (147.1, 113.1), turned to 90 degrees
- moved C114 45.8 mm to (149.4, 113.0), turned to 90 degrees
- moved SW101 37.8 mm to (160.3, 113.1), turned to -90 degrees
- moved C302 32.4 mm to (181.1, 149.1)
- moved C301 32.4 mm to (186.4, 144.3)
- moved R301 32.4 mm to (185.2, 147.3)
- moved U303 32.4 mm to (182.9, 144.2)
- moved R113 31.5 mm to (134.6, 114.7)
- moved R103 31.3 mm to (134.6, 113.5), turned to 180 degrees
- moved C101 29.1 mm to (133.9, 115.0), turned to -90 degrees
- moved J104 25.3 mm to (167.8, 99.7), turned to 90 degrees
- moved C104 21.7 mm to (128.3, 114.7), turned to 180 degrees
- moved C108 18.2 mm to (132.3, 102.9), turned to 0 degrees
- moved C106 17.4 mm to (125.5, 102.1), turned to 180 degrees
- moved C105 15.7 mm to (121.8, 113.3), turned to 90 degrees
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Routing:
- net GNDD: track 100.6 -> 117.3 mm, vias 22 -> 27
- net /USART1_TX: track 1.32 -> 14.8 mm, vias 0 -> 1
- net Net-(SW101-A): track 0.00 -> 11.8 mm
- net /TX_LED: track 3.84 -> 15.2 mm, vias 0 -> 1
- net /USART1_RX: track 0.00 -> 10.4 mm, vias 0 -> 1
- net /SPI2_MISO: track 0.00 -> 9.93 mm
- net /SPI2_SCK: track 0.00 -> 9.12 mm
- net /5V_USB: track 29.4 -> 21.1 mm
- net /SPI2_NSS: track 0.00 -> 5.22 mm
- net /SPI2_MOSI: track 0.00 -> 4.99 mm
- net Net-(U102-3V3OUT): track 0.00 -> 4.07 mm
- net Net-(U103-EN): track 8.03 -> 4.30 mm
- net Net-(U102-CBUS0): track 0.00 -> 3.38 mm
- net +3V3: track 38.7 -> 42.0 mm, vias 10 -> 12
- net +5V: track 18.3 -> 21.0 mm, vias 0 -> 1
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- removed copper zone on In2.Cu, net +3V3
- removed copper zone on In1.Cu, net GNDD
